File: hardware/esp-dht/esp-dht.sch (KiCad schematic (older format))
At the start: 3 parts, among them J1 Conn_01x02_Male, U1 L78L33_TO220

Commit message: complete kicad schematic and gitignore kicad caches
Parts:
- removed U1: L78L33_TO220, Package_TO_SOT_THT:TO-220-3_Vertical, symbol Regulator_Linear:L78L33_TO92
- added J2: FTDI Header pt 1, symbol Connector:Conn_01x03_Male
- added J3: FTDI Header pt 2, symbol Connector:Conn_01x01_Male
- added U1: ESP-01v090, symbol ESP8266:ESP-01v090
- added U3: LD1117v33, symbol Regulator_Linear:AZ1117-3.3
- J1: value Conn_01x02_Male -> PWR IN
- gave numbers to parts that had none: 1
Connections:
- net +3V3: now also J2.1 (Pin_1), U1.3 (CH_PD), U1.5 (RST), U1.7 (VCC), U3.2 (VO)
- net +BATT: now also U3.3 (VI)
- net Earth: now also J3.1 (Pin_1), U1.2 (GND), U3.1 (GND)
- net DATA: now reaches U2.2 (IO)
- net DATA: now also U1.6 (GPIO0)
- new net ESP_RX: J2.2 (Pin_2), U1.8 (URXD)
- new net ESP_TX: J2.3 (Pin_3), U1.1 (UTXD)
Other:
- moved on the sheet: J1, U2
